Commit message: implemented pointclud assembly and publishing

File: urdf/3d_scanner.urdf (robot description, URDF)
Before this commit: robot laser_halterung, 8 links, 7 joints
Links:
- removed link laser360
- added link laser; collision mesh filename=package://uos_common_urdf/meshes/sick_lms-200.stl; visual mesh filename=package://uos_common_urdf/meshes/sick_lms-200.stl
Joints:
- joint laser_to_halterung: child laser360 -> laser
